File: Motherboard/_autosave-mainboard.sch (KiCad schematic (older format))
At the start: 50 parts, among them IC1 BMX160, J1 Conn_01x01, J2 10118194-0001LF, J28 Conn_01x01, J29 Conn_01x01, J3 Micro_SD_Card, J30 Conn_01x01, J4 xf2m-2415-1a, J5 XF2M-1015-1A, J6 U.FL-R-SMT-1, J7 U.FL-R-SMT-1, J8 Conn_01x01, SW1 KMR231NG LFS, U1 RFM95W-915S2, U2 ATSAMD51G_TQFN48, U3 DRV8848, U4 TPS82740BSIPR, U5 DRV8848, U6 MAX708RESA-T, U8 RFM95W-915S2

Commit message: placement getting closer
Connections:
- net CS_RF1 is gone; now on net RF1_CS: U8.5 (NSS)
- net CS_RF2 is gone; now on net RF2_CS: U1.5 (NSS)
- net RF_BUSY is gone; now on net RF1_BUSY: U8.12 (DIO4)
- net RF_DIO1 is gone; now on net RF1_IO1: U8.15 (DIO1)
- net RF_RST is gone; now on net RF1_RST: U8.6 (RESET)
- net CS_CAM: no longer U2.24 (PA15/I15/SERCOM2+4.3)
- net CS_IMU: no longer U2.27 (PA18/I2/SERCOM1+3.2)
- net EN_CAM: no longer U2.29 (PA20/I4/SERCOM3+5.2/I2SFS0)
- net RF2_IO1: now also U1.15 (DIO1)
- net SCL2: now also J4.2; no longer J4.1
- net SDA2: now also J4.1; no longer J4.2
- net RF_DIO0: no longer names the net of U8.14 (DIO0)
- net RF_DIO2: no longer names the net of U8.16 (DIO2)
- net RF_DIO3: no longer names the net of U8.11 (DIO3)
Changed lines of the file:
@@
 Wire Wire Line
 	7750 5350 7850 5350
-Wire Wire Line
-	8850 5650 8950 5650
-Text GLabel 8950 5650 2    50   BiDi ~ 0
-RF_DIO2
 $Comp
 L power:GND #PWR0140
@@
 Wire Wire Line
 	7850 5650 7750 5650
-Text GLabel 7750 5450 0    50   Input ~ 0
-CS_RF1
-Text GLabel 7750 5650 0    50   BiDi ~ 0
-RF_RST
-Text GLabel 8950 5550 2    50   BiDi ~ 0
-RF_DIO3
-Text GLabel 8950 5450 2    50   Output ~ 0
-RF_BUSY
-Text GLabel 8950 5750 2    50   BiDi ~ 0
-RF_DIO1
-Wire Wire Line
-	8950 5550 8850 5550
-Wire Wire Line
-	8950 5750 8850 5750
 Wire Wire Line
 	8950 5450 8850 5450
-Text GLabel 8950 5850 2    50   BiDi ~ 0
-RF_DIO0
-Wire Wire Line
-	8950 5850 8850 5850
 Text GLabel 4600 4500 2    50   BiDi ~ 0
 DAC1
@@
 $EndComp
 Wire Wire Line
-	8900 4200 8800 4200
-Wire Wire Line
 	8900 4400 8800 4400
-Text GLabel 8800 4200 0    50   Input ~ 0
-CS_RF2
 Text GLabel 8800 4400 0    50   BiDi ~ 0
 RF2_RST
@@
 Text GLabel 5950 3050 2    50   Input ~ 0
 BATT_N
-Text GLabel 4550 5700 2    50   Input ~ 0
+Text GLabel -1100 4600 2    50   Input ~ 0
 CS_CAM
 Connection ~ 1450 7000
@@
 	1    0    0    -1
 $EndComp
-Text GLabel 4550 6200 2    50   Input ~ 0
+Text GLabel -1050 4400 2    50   Input ~ 0
 EN_CAM
 Text GLabel 5300 5800 2    59   BiDi ~ 0
@@
 Text GLabel 4700 4100 2    59   BiDi ~ 0
 SCL1
-Wire Wire Line
-	4550 5700 4450 5700
 Text Notes 1650 7550 0    50   ~ 0
 UART:\nTX: PB08\nRX: PB09\n
@@
 Text GLabel 5200 1950 0    59   BiDi ~ 0
 SCL1
+Text GLabel 6100 1250 2    59   BiDi ~ 0
+SCL2
 Text GLabel 5200 1250 0    59   BiDi ~ 0
-SCL2
-Text GLabel 6100 1250 2    59   BiDi ~ 0
 SDA2
-Wire Wire Line
-	4550 6200 4450 6200
 $Comp
 L mainboard-rescue:R_US-Device R4
@@
 Wire Wire Line
 	5250 5800 5300 5800
-Text GLabel 4450 6000 2    50   Output ~ 0
-CS_IMU
 $Comp
 L mainboard-rescue:XF2M-1015-1A-symbols J5
@@
 Wire Wire Line
 	4650 7350 4700 7350
-Text GLabel -3900 5050 0    50   Input ~ 0
+Text GLabel -1750 5200 0    50   Input ~ 0
 DXZ_FAULT
-Text GLabel -3900 5150 0    50   Input ~ 0
+Text GLabel -1750 5300 0    50   Input ~ 0
 MXZ_EN
-Text GLabel -3900 5350 0    50   Input ~ 0
+Text GLabel -1750 5500 0    50   Input ~ 0
 MINX_1
-Text GLabel -3900 5450 0    50   Input ~ 0
+Text GLabel -1750 5600 0    50   Input ~ 0
 MINX_2
-Text GLabel -3900 5650 0    50   Input ~ 0
+Text GLabel -1750 5800 0    50   Input ~ 0
 MINZ_1
-Text GLabel -3900 5750 0    50   Input ~ 0
+Text GLabel -1750 5900 0    50   Input ~ 0
 MINZ_2
-Text GLabel -3400 5050 0    50   Input ~ 0
+Text GLabel -1250 5200 0    50   Input ~ 0
 DY_FAULT
-Text GLabel -3400 5150 0    50   Input ~ 0
+Text GLabel -1250 5300 0    50   Input ~ 0
 MY_EN
-Text GLabel -3400 5350 0    50   Input ~ 0
+Text GLabel -1250 5500 0    50   Input ~ 0
 MINY_1
-Text GLabel -3400 5450 0    50   Input ~ 0
+Text GLabel -1250 5600 0    50   Input ~ 0
 MINY_2
 $Comp
@@
 Text GLabel -2050 6450 2    50   BiDi ~ 0
 RF1_BUSY
+Text GLabel -2050 6550 2    50   BiDi ~ 0
+RF1_RST
+Text GLabel -2050 6650 2    50   BiDi ~ 0
+RF1_CS
+Text GLabel -1550 6450 2    50   BiDi ~ 0
+RF1_IO1
+Text GLabel 8800 4200 0    50   BiDi ~ 0
+RF2_CS
+Wire Wire Line
+	8800 4200 8900 4200
+Text GLabel -2050 6100 2    50   BiDi ~ 0
+RF2_CS
+Text GLabel -1550 6300 2    50   BiDi ~ 0
+RF2_IO1
+Text GLabel -2050 6200 2    50   BiDi ~ 0
+RF2_RST
 Text GLabel -2050 6300 2    50   BiDi ~ 0
 RF2_BUSY
-Text GLabel -2050 6550 2    50   BiDi ~ 0
+Text GLabel 10000 4500 2    50   BiDi ~ 0
+RF2_IO1
+Wire Wire Line
+	10000 4500 9900 4500
+Text GLabel 8950 5450 2    50   BiDi ~ 0
+RF1_BUSY
+Text GLabel 7750 5650 0    50   BiDi ~ 0
 RF1_RST
-Text GLabel -2050 6200 2    50   BiDi ~ 0
-RF2_RST
-Text GLabel -2050 6650 2    50   BiDi ~ 0
+Text GLabel 7750 5450 0    50   BiDi ~ 0
 RF1_CS
-Text GLabel -2050 6100 2    50   BiDi ~ 0
-RF2_CS
-Text GLabel -1550 6450 2    50   BiDi ~ 0
+Text GLabel 8950 5750 2    50   BiDi ~ 0
 RF1_IO1
-Text GLabel -1550 6300 2    50   BiDi ~ 0
-RF2_IO1
+Wire Wire Line
+	8950 5750 8850 5750
+Text GLabel -1100 4850 2    50   Output ~ 0
+CS_IMU
 $EndSCHEMATC
