File: Motherboard/mainboard.sch (KiCad schematic (older format))
At the start: 57 parts, among them IC1 BMX160, J1 Conn_01x01, J2 10118194-0001LF, J28 Conn_01x01, J29 Conn_01x01, J3 Micro_SD_Card, J30 Conn_01x01, J4 xf2m-2415-1a, J5 XF2M-1015-1A, J6 U.FL-R-SMT-1, J7 U.FL-R-SMT-1, J8 Conn_01x01, SW1 KMR231NG LFS, U1 RFM95W-915S2, U2 ATSAMD51G_TQFN48, U3 DRV8848, U4 TPS82740BSIPR, U5 DRV8848, U6 MAX708RESA-T, U8 RFM95W-915S2

Commit message: 100% routed
Parts:
- removed J1, J28, J29, J30, J8: Conn_01x01, TestPoint:TestPoint_Pad_D1.0mm, symbol mainboard-rescue:Conn_01x01-Connector_Generic
- added J1: Conn_01x06, Connector_PinHeader_1.27mm:PinHeader_2x03_P1.27mm_Vertical_SMD, symbol Connector_Generic:Conn_01x06
- added J9: Conn_01x02, Connector_PinHeader_2.54mm:PinHeader_1x02_P2.54mm_Vertical, symbol Connector_Generic:Conn_01x02
Connections:
- net BATT_N is gone; now on net GND: J5.4
- net +3V3: now also J1.1 (Pin_1)
- net BATT_P: now also J9.2 (Pin_2)
- net CS_CAM: now also J5.9; no longer J5.6
- net EN_CAM: now also J5.8; no longer J5.5
- net GND: now also J1.3 (Pin_3), J9.1 (Pin_1)
- net MOSI: now also J5.5; no longer J5.8
- net SCK: now also J5.6; no longer J5.9
- net SWCLK: now also J1.4 (Pin_4)
- net SWDIO: now also J1.2 (Pin_2)
- net ~RESET: now also J1.5 (Pin_5)
Changed lines of the file:
@@
 	5300 7100 5300 7200
 Wire Wire Line
-	4900 7200 4900 7350
+	4900 7200 4900 7500
 $Comp
 L mainboard-rescue:CAP_CERAMIC0603_NO- C?
@@
 Connection ~ 5000 7200
 Wire Wire Line
-	5000 7200 5000 7350
-Wire Wire Line
 	5350 4550 5350 4750
 Wire Wire Line
@@
 L power:+3V3 #PWR0116
 U 1 1 5D84CDF6
-P 4800 7350
-F 0 "#PWR0116" H 4800 7200 50  0001 C CNN
-F 1 "+3V3" H 4815 7523 50  0000 C CNN
-F 2 "" H 4800 7350 50  0001 C CNN
-F 3 "" H 4800 7350 50  0001 C CNN
-	1    4800 7350
+P 4600 7400
+F 0 "#PWR0116" H 4600 7250 50  0001 C CNN
+F 1 "+3V3" H 4750 7450 50  0000 C CNN
+F 2 "" H 4600 7400 50  0001 C CNN
+F 3 "" H 4600 7400 50  0001 C CNN
+	1    4600 7400
 	1    0    0    -1
 $EndComp
@@
 Text GLabel 4600 4500 2    50   Input ~ 0
 BATTERY
-$Comp
-L mainboard-rescue:Conn_01x01-Connector_Generic J28
-U 1 1 5D2A6718
-P 5000 7550
-F 0 "J28" V 5100 7450 50  0000 L CNN
-F 1 "Conn_01x01" V 4963 7630 50  0001 L CNN
-F 2 "TestPoint:TestPoint_Pad_D1.0mm" H 5000 7550 50  0001 C CNN
-F 3 "~" H 5000 7550 50  0001 C CNN
-F 4 "DNP" H 0   0   50  0001 C CNN "DNP"
-	1    5000 7550
-	0    1    1    0
-$EndComp
-$Comp
-L mainboard-rescue:Conn_01x01-Connector_Generic J1
-U 1 1 5D2B62DF
-P 4900 7550
-F 0 "J1" V 5000 7500 50  0000 L CNN
-F 1 "Conn_01x01" V 4863 7630 50  0001 L CNN
-F 2 "TestPoint:TestPoint_Pad_D1.0mm" H 4900 7550 50  0001 C CNN
-F 3 "~" H 4900 7550 50  0001 C CNN
-F 4 "DNP" H 0   0   50  0001 C CNN "DNP"
-	1    4900 7550
-	0    1    1    0
-$EndComp
-$Comp
-L mainboard-rescue:Conn_01x01-Connector_Generic J29
-U 1 1 5D32C3EB
-P 4800 7550
-F 0 "J29" V 4900 7450 50  0000 L CNN
-F 1 "Conn_01x01" V 4763 7630 50  0001 L CNN
-F 2 "TestPoint:TestPoint_Pad_D1.0mm" H 4800 7550 50  0001 C CNN
-F 3 "~" H 4800 7550 50  0001 C CNN
-F 4 "DNP" H 0   0   50  0001 C CNN "DNP"
-	1    4800 7550
-	0    1    1    0
-$EndComp
-$Comp
-L mainboard-rescue:Conn_01x01-Connector_Generic J30
-U 1 1 5D338152
-P 5100 7550
-F 0 "J30" V 5200 7500 50  0000 L CNN
-F 1 "Conn_01x01" V 5063 7630 50  0001 L CNN
-F 2 "TestPoint:TestPoint_Pad_D1.0mm" H 5100 7550 50  0001 C CNN
-F 3 "~" H 5100 7550 50  0001 C CNN
-F 4 "DNP" H 0   0   50  0001 C CNN "DNP"
-	1    5100 7550
-	0    1    1    0
-$EndComp
 Wire Wire Line
 	5700 5350 5700 5550
@@
 L power:GND #PWR0139
 U 1 1 5DB21F1D
-P 5350 7350
-F 0 "#PWR0139" H 5350 7100 50  0001 C CNN
-F 1 "GND" H 5355 7177 50  0000 C CNN
-F 2 "" H 5350 7350 50  0001 C CNN
-F 3 "" H 5350 7350 50  0001 C CNN
-	1    5350 7350
-	1    0    0    -1
+P 4650 7600
+F 0 "#PWR0139" H 4650 7350 50  0001 C CNN
+F 1 "GND" V 4650 7400 50  0000 C CNN
+F 2 "" H 4650 7600 50  0001 C CNN
+F 3 "" H 4650 7600 50  0001 C CNN
+	1    4650 7600
+	0    -1   -1   0
 $EndComp
 $Comp
@@
 	5850 7350 5350 7350
 Connection ~ 5350 7350
-Wire Wire Line
-	5100 7350 5350 7350
-Wire Wire Line
-	5350 7000 5350 7350
 $Comp
 L mainboard-rescue:C-Device C9
@@
 Text GLabel 10000 1700 2    50   Input ~ 0
 MOY_2
-Text GLabel 6300 1050 2    50   Output ~ 0
+Text GLabel 5400 950  0    50   Output ~ 0
 MOSI
 Text GLabel 5400 1050 0    50   Input ~ 0
 MISO
+Text GLabel 6300 950  2    50   Input ~ 0
+SCK
+Text GLabel 6300 1050 2    50   Input ~ 0
+EN_CAM
 Text GLabel 5400 1150 0    50   Input ~ 0
-SCK
-Text GLabel 5400 950  0    50   Input ~ 0
-EN_CAM
-Text GLabel 6300 750  2    50   Input ~ 0
-GND
-Text GLabel 6300 950  2    50   Input ~ 0
 CS_CAM
-Text GLabel 6300 850  2    50   Input ~ 0
-BATT_N
 Text GLabel 1450 5800 0    50   Output ~ 0
 CS_CAM
@@
 	1    0    0    -1
 $EndComp
-$Comp
-L mainboard-rescue:Conn_01x01-Connector_Generic J8
-U 1 1 5DC2AE71
-P 4700 7550
-F 0 "J8" V 4800 7450 50  0000 L CNN
-F 1 "Conn_01x01" V 4663 7630 50  0001 L CNN
-F 2 "TestPoint:TestPoint_Pad_D1.0mm" H 4700 7550 50  0001 C CNN
-F 3 "~" H 4700 7550 50  0001 C CNN
-F 4 "DNP" H -300 0   50  0001 C CNN "DNP"
-	1    4700 7550
-	0    1    1    0
-$EndComp
-Text GLabel 4650 7350 0    50   BiDi ~ 0
+Text GLabel 4700 7800 2    50   BiDi ~ 0
 ~RESET
-Wire Wire Line
-	4650 7350 4700 7350
 Text GLabel 4450 5600 2    50   Output ~ 0
 MINX_1
@@
 Text Notes 7950 3950 2    50   ~ 0
 X
-Wire Wire Line
-	7400 4050 7000 4050
 Text Label 7050 3950 0    50   ~ 0
 MOZ_1
@@
 	0    1    1    0
 $EndComp
+Wire Wire Line
+	7000 4050 7400 4050
+$Comp
+L Connector_Generic:Conn_01x02 J9
+U 1 1 5DB310E1
+P 7100 4350
+F 0 "J9" H 7018 4025 50  0000 C CNN
+F 1 "Conn_01x02" H 7018 4116 50  0000 C CNN
+F 2 "Connector_PinHeader_2.54mm:PinHeader_1x02_P2.54mm_Vertical" H 7100 4350 50  0001 C CNN
+F 3 "~" H 7100 4350 50  0001 C CNN
+	1    7100 4350
+	-1   0    0    1
+$EndComp
+Text GLabel 7400 4250 2    50   Input ~ 0
+BATT_P
+Wire Wire Line
+	7300 4250 7400 4250
+$Comp
+L power:GND #PWR0150
+U 1 1 5DB3B3E4
+P 7400 4350
+F 0 "#PWR0150" H 7400 4100 50  0001 C CNN
+F 1 "GND" H 7405 4177 50  0000 C CNN
+F 2 "" H 7400 4350 50  0001 C CNN
+F 3 "" H 7400 4350 50  0001 C CNN
+	1    7400 4350
+	1    0    0    -1
+$EndComp
+Wire Wire Line
+	7400 4350 7300 4350
+$Comp
+L power:GND #PWR0151
+U 1 1 5DB658C1
+P 6400 750
+F 0 "#PWR0151" H 6400 500 50  0001 C CNN
+F 1 "GND" H 6550 700 50  0000 C CNN
+F 2 "" H 6400 750 50  0001 C CNN
+F 3 "" H 6400 750 50  0001 C CNN
+	1    6400 750
+	1    0    0    -1
+$EndComp
+Wire Wire Line
+	6400 750  6300 750
+Wire Wire Line
+	6300 750  6300 850
+Connection ~ 6300 750
+$Comp
+L Connector_Generic:Conn_01x06 J1
+U 1 1 5DB917BE
+P 4400 7600
+F 0 "J1" H 4400 7900 50  0000 C CNN
+F 1 "Conn_01x06" V 4500 7600 50  0000 C CNN
+F 2 "Connector_PinHeader_1.27mm:PinHeader_2x03_P1.27mm_Vertical_SMD" H 4400 7600 50  0001 C CNN
+F 3 "~" H 4400 7600 50  0001 C CNN
+	1    4400 7600
+	-1   0    0    -1
+$EndComp
+Wire Wire Line
+	5350 7000 5350 7350
+Wire Wire Line
+	4700 7800 4600 7800
+Wire Wire Line
+	5200 7600 5200 7350
+Wire Wire Line
+	5200 7350 5350 7350
+Wire Wire Line
+	4900 7500 4600 7500
+Wire Wire Line
+	4650 7600 4600 7600
+Wire Wire Line
+	5000 7700 4600 7700
+Wire Wire Line
+	5000 7200 5000 7700
+$Comp
+L power:GND #PWR0152
+U 1 1 5DC68C68
+P 5200 7600
+F 0 "#PWR0152" H 5200 7350 50  0001 C CNN
+F 1 "GND" V 5200 7400 50  0000 C CNN
+F 2 "" H 5200 7600 50  0001 C CNN
+F 3 "" H 5200 7600 50  0001 C CNN
+	1    5200 7600
+	1    0    0    -1
+$EndComp
 $EndSCHEMATC

Commit message: finished- might fiddle with later
Parts:
- renumbered IC1 to U7
Changed lines of the file:
@@
 	5700 5350 5700 5550
 $Comp
-L mainboard-rescue:BMX160-symbols IC1
+L mainboard-rescue:BMX160-symbols U7
 U 1 1 5DAD1297
 P 1300 1000
-F 0 "IC1" H 1900 1265 50  0000 C CNN
+F 0 "U7" H 1900 1265 50  0000 C CNN
 F 1 "BMX160" H 1900 1174 50  0000 C CNN
 F 2 "custom-footprints:BMX160" H 2350 1100 50  0001 L CNN
