File: rf-test/spriteSAMD.kicad_pcb (KiCad board)
At the start: 2 copper layers, 25.7 x 29.8 mm, 7 parts, among them J1 Conn_01x08_Female, J2 Conn_Coaxial, J3 Conn_01x08_Female, U1 RFM95W-915S2

Commit message: rftest ready for fab
Routing:
- net GND: vias 21 -> 22
- net (no net): vias 1 -> 0
Changed lines of the file:
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@@
   )
   (setup
-    (last_trace_width 0.6)
+    (last_trace_width 0.0889)
     (user_trace_width 0.0889)
     (user_trace_width 0.127)
@@
     (descr "Through hole straight pin header, 1x06, 2.54mm pitch, single row")
     (tags "Through hole pin header THT 1x06 2.54mm single row")
-    (fp_text reference J3 (at 0 -2.33 90) (layer F.SilkS)
+    (fp_text reference J3 (at 0 -2.33 90) (layer F.SilkS) hide
       (effects (font (size 1 1) (thickness 0.15)))
     )
@@
     (tags SMA)
     (attr smd)
-    (fp_text reference J2 (at -3.5 0) (layer F.SilkS)
+    (fp_text reference J2 (at -3.5 0) (layer F.SilkS) hide
       (effects (font (size 1 1) (thickness 0.15)))
     )
@@
     (descr "Through hole straight pin header, 1x08, 2.54mm pitch, single row")
     (tags "Through hole pin header THT 1x08 2.54mm single row")
-    (fp_text reference J1 (at 0 -2.33 90) (layer F.SilkS)
+    (fp_text reference J1 (at 0 -2.33 90) (layer F.SilkS) hide
       (effects (font (size 1 1) (thickness 0.15)))
     )
@@
   (gr_line (start 171.704 65.9384) (end 171.704 95.7072) (layer Edge.Cuts) (width 0.1))
   (gr_line (start 170.4086 65.9384) (end 171.704 65.9384) (layer Edge.Cuts) (width 0.1))
-  (via (at 168.3258 67.5894) (size 0.45) (drill 0.3) (layers Top Bottom) (net 0))
+  (via (at 168.3258 67.5894) (size 0.45) (drill 0.3) (layers Top Bottom) (net 1))
   (segment (start 166.893 91.709) (end 168.7322 93.5482) (width 0.3302) (layer Top) (net 1))
   (segment (start 166.893 88.6466) (end 166.893 91.709) (width 0.3302) (layer Top) (net 1))
@@
   (zone (net 1) (net_name GND) (layer Top) (hatch edge 0.508)
     (connect_pads (clearance 0.127))
-    (min_thickness 0.254)
-    (fill yes (arc_segments 32) (thermal_gap 0.508) (thermal_bridge_width 0.508))
+    (min_thickness 0.127)
+    (fill yes (arc_segments 32) (thermal_gap 0.127) (thermal_bridge_width 0.381))
     (polygon
       (pts
@@
   (zone (net 1) (net_name GND) (layer Bottom) (hatch edge 0.508)
     (connect_pads (clearance 0.127))
-    (min_thickness 0.254)
-    (fill yes (arc_segments 32) (thermal_gap 0.508) (thermal_bridge_width 0.508))
+    (min_thickness 0.127)
+    (fill yes (arc_segments 32) (thermal_gap 0.127) (thermal_bridge_width 0.381))
     (polygon
       (pts
